File: eRIC_breakout.brd (EAGLE design)
At the start: 19.8 x 68.1 mm, 30 parts

Commit message: BOM, component names and values
Parts:
- renumbered E$2 to C1, E$3 to SMA, E$4 to R2, E$9 to R1
Changed lines of the file:
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@@
 <element name="E$29" library="testpad" package="TP11R" value="" x="25.35" y="42.05"/>
 <element name="E$8" library="adafruit" package="1X12-CB" value="" x="14" y="19.8" rot="R90"/>
-<element name="E$3" library="SparkFun-Connectors" package="SMA-EDGE" value="" x="12.7" y="67.7"/>
+<element name="SMA" library="SparkFun-Connectors" package="SMA-EDGE" value="" x="12.7" y="67.7"/>
 <element name="E$1" library="adafruit" package="1X12-CB" value="" x="26.7" y="19.85" rot="R90"/>
-<element name="E$2" library="eagle-ltspice" package="C0603" value="" x="16.225" y="19.825" rot="MR90"/>
-<element name="E$4" library="eagle-ltspice" package="R0402" value="" x="16.15" y="27" rot="MR90"/>
-<element name="E$9" library="eagle-ltspice" package="R0402" value="" x="16.125" y="30.7" rot="MR270"/>
+<element name="C1" library="eagle-ltspice" package="C0603" value="" x="16.225" y="19.825" rot="MR90"/>
+<element name="R2" library="eagle-ltspice" package="R0402" value="" x="16.15" y="27" rot="MR90"/>
+<element name="R1" library="eagle-ltspice" package="R0402" value="" x="16.125" y="30.7" rot="MR270"/>
 </elements>
 <signals>
@@
 <wire x1="13.9" y1="41.82605" x2="13.9" y2="45.9" width="0.4064" layer="1"/>
 <wire x1="13.9" y1="45.9" x2="12.65" y2="47.15" width="0.4064" layer="1" curve="90"/>
-<contactref element="E$2" pad="2"/>
+<contactref element="C1" pad="2"/>
 <wire x1="16.75" y1="37" x2="16.75" y2="37.05" width="0.254" layer="1"/>
 <wire x1="16.225" y1="20.675" x2="15.845" y2="21.07" width="0.3048" layer="16"/>
@@
 </polygon>
 <contactref element="E$12" pad="TP"/>
-<contactref element="E$3" pad="GND@0"/>
-<contactref element="E$3" pad="GND@1"/>
+<contactref element="SMA" pad="GND@0"/>
+<contactref element="SMA" pad="GND@1"/>
 <via x="13.65" y="64.45" extent="1-16" drill="0.3"/>
 <via x="13.65" y="63.3" extent="1-16" drill="0.3"/>
@@
 </polygon>
 <contactref element="E$1" pad="12"/>
-<contactref element="E$3" pad="GND@3"/>
-<contactref element="E$3" pad="GND@2"/>
-<contactref element="E$2" pad="1"/>
+<contactref element="SMA" pad="GND@3"/>
+<contactref element="SMA" pad="GND@2"/>
+<contactref element="C1" pad="1"/>
 </signal>
 <signal name="S$26">
-<contactref element="E$9" pad="2"/>
+<contactref element="R1" pad="2"/>
 <contactref element="E$8" pad="10"/>
 <wire x1="16.125" y1="30.05" x2="14.765" y2="28.69" width="0.254" layer="16"/>
@@
 <via x="16.35" y="54.8" extent="1-16" drill="0.3"/>
 <wire x1="16.35" y1="54.8" x2="12.65" y2="54.8" width="0.254" layer="1"/>
-<contactref element="E$9" pad="1"/>
+<contactref element="R1" pad="1"/>
 <wire x1="16.35" y1="31.575" x2="16.125" y2="31.35" width="0.254" layer="16"/>
 </signal>
@@
 </signal>
 <signal name="S$25">
-<contactref element="E$3" pad="SIG"/>
+<contactref element="SMA" pad="SIG"/>
 <contactref element="E$11" pad="TP"/>
 <wire x1="15.2" y1="62.45" x2="15.24" y2="62.54656875" width="0.6096" layer="1" curve="45"/>
@@
 <signal name="S$2">
 <contactref element="TX" pad="TP"/>
-<contactref element="E$4" pad="2"/>
+<contactref element="R2" pad="2"/>
 <wire x1="12.65" y1="52.3" x2="17.15" y2="52.3" width="0.254" layer="1"/>
 <via x="17.15" y="52.3" extent="1-16" drill="0.3"/>
@@
 <signal name="S$4">
 <contactref element="E$8" pad="9"/>
-<contactref element="E$4" pad="1"/>
+<contactref element="R2" pad="1"/>
 <wire x1="16.15" y1="26.35" x2="16.025" y2="26.15" width="0.254" layer="16"/>
 <wire x1="16.025" y1="26.15" x2="14" y2="26.15" width="0.254" layer="16"/>

Commit message: component values
Parts:
- C1: value (none) -> .1uF
- R1, R2: value (none) -> 10k
Changed lines of the file:
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@@
 <element name="SMA" library="SparkFun-Connectors" package="SMA-EDGE" value="" x="12.7" y="67.7"/>
 <element name="E$1" library="adafruit" package="1X12-CB" value="" x="26.7" y="19.85" rot="R90"/>
-<element name="C1" library="eagle-ltspice" package="C0603" value="" x="16.225" y="19.825" rot="MR90"/>
-<element name="R2" library="eagle-ltspice" package="R0402" value="" x="16.15" y="27" rot="MR90"/>
-<element name="R1" library="eagle-ltspice" package="R0402" value="" x="16.125" y="30.7" rot="MR270"/>
+<element name="C1" library="eagle-ltspice" package="C0603" value=".1uF" x="16.225" y="19.825" rot="MR90"/>
+<element name="R2" library="eagle-ltspice" package="R0402" value="10k" x="16.15" y="27" rot="MR90"/>
+<element name="R1" library="eagle-ltspice" package="R0402" value="10k" x="16.125" y="30.7" rot="MR270"/>
 </elements>
 <signals>

Commit message: overhaul of design, include schematic, un-tested
Parts:
- removed E$1, E$8: (no value), adafruit:1X12-CB
- removed E$10, E$11, E$12, E$13, E$14, E$15, E$16, E$17, E$18, E$19, E$20, E$21, E$22, E$25, E$27, E$28, E$29, E$6, E$7, GND, RESET, RX, TX, VCC: (no value), testpad:TP11R
- removed SMA: (no value), SparkFun-Connectors:SMA-EDGE
- added H1, H2: (no value), SparkFun-Connectors:1X12_NO_SILK_KIT
- added J$1: SMA_EDGE, SparkFun-Connectors:SMA-EDGE
- added U1: ERIC, lprs:ERIC
- C1: value .1uF -> (none); device eagle-ltspice:C0603 -> adafruit:C0603K
- R1, R2: value 10k -> (none); device eagle-ltspice:R0402 -> adafruit:R0603
- moved C1 11.0 mm to (5.40, 18.1)
- moved R2 10.8 mm to (5.42, 25.4), turned to 270 degrees
- moved R1 10.8 mm to (5.40, 29.5)
Connections:
- removed net S$1: C1.2, E$8.7, VCC.TP
- removed net S$10: E$6.TP, E$8.12
- removed net S$11: E$7.TP, E$8.11
- removed net S$12: E$10.TP, E$8.8
- removed net S$13: E$1.3, E$22.TP
- removed net S$14: E$1.2, E$21.TP
- removed net S$15: E$1.4, E$20.TP
- removed net S$16: E$1.5, E$19.TP
- removed net S$17: E$1.6, E$18.TP
- removed net S$18: E$1.7, E$17.TP
- removed net S$19: E$1.8, E$16.TP
- removed net S$2: R2.2, TX.TP
- removed net S$20: R1.1, RX.TP
- removed net S$21: E$28.TP, E$8.2
- removed net S$22: E$27.TP, E$8.3
- removed net S$23: E$25.TP, E$8.5
- removed net S$24: E$29.TP, E$8.1
- removed net S$25: E$11.TP, SMA.SIG
- removed net S$26: E$8.10, R1.2
- removed net S$3: E$8.4, RESET.TP
- removed net S$4: E$8.9, R2.1
- removed net S$6: E$1.11, E$13.TP
- removed net S$7: E$1.10, E$14.TP
- removed net S$9: E$1.9, E$15.TP
- new net N$1: H1.1, U1.CD
- new net N$11: H1.8, U1.E8
- new net N$12: H1.9, U1.E9
- new net N$13: H1.10, U1.E10
- new net N$14: H1.11, U1.E11
- new net N$15: H1.12, U1.E12
- new net N$16: H2.9, U1.E15
- new net N$17: H2.8, U1.E16
- new net N$18: H2.7, U1.E17
- new net N$19: H2.6, U1.E18
- new net N$2: H1.2, U1.BUSY
- new net N$20: H2.5, U1.E19
- new net N$21: H2.4, U1.E20
- new net N$22: H2.3, U1.E21
- new net N$23: H2.2, U1.E22
- new net N$24: H2.11, U1.FS
- new net N$25: H2.10, U1.E13
- new net N$3: J$1.SIG, U1.ANT
- new net N$8: H1.5, U1.HR
- new net SDI: H1.4, R2.1, R2.2, U1.SDI
- new net SDO: H1.3, R1.1, R1.2, U1.SDO
- new net VCC: C1.2, H1.6, U1.VCC
- net GND: now also H1.7, H2.1, H2.12, J$1.GND@0, J$1.GND@1, J$1.GND@2, J$1.GND@3, U1.AGND, U1.GND; no longer E$1.1, E$1.12, E$12.TP, E$8.6, GND.TP, SMA.GND@0, SMA.GND@1, SMA.GND@2, SMA.GND@3
Routing:
- net N$16: track 0.00 -> 50.9 mm, vias 0 -> 1
- net S$15: track 50.2 -> 0.00 mm, vias 1 -> 0
- net N$17: track 0.00 -> 49.2 mm, vias 0 -> 1
- net S$16: track 48.4 -> 0.00 mm, vias 1 -> 0
- net N$18: track 0.00 -> 47.6 mm, vias 0 -> 1
- net S$17: track 46.7 -> 0.00 mm, vias 1 -> 0
- net N$19: track 0.00 -> 46.0 mm, vias 0 -> 1
- net S$18: track 44.9 -> 0.00 mm, vias 1 -> 0
- net N$15: track 0.00 -> 43.7 mm
- net S$19: track 43.0 -> 0.00 mm, vias 1 -> 0
- net S$24: track 42.2 -> 0.00 mm
- net N$24: track 0.00 -> 41.7 mm
- net N$21: track 0.00 -> 40.7 mm, vias 0 -> 2
- net S$14: track 40.5 -> 0.00 mm
- net N$14: track 0.00 -> 40.0 mm
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Other:
- board size 19.8 x 68.1 mm -> 21 x 69 mm
- board text added: "APR:H06"
- board text removed: "JUN:S05"

Commit message: v1.6 ordered 4/18/2015
Parts:
- removed U1: ERIC, lprs:ERIC
- added IC1: ERIC, lprs:ERIC
- H1, H2: device SparkFun-Connectors:1X12_NO_SILK_KIT -> adafruit:1X12-CB
- moved H1 13.2 mm to (4.64, 18.7)
- moved H2 13.2 mm to (19.9, 18.7)
- moved C1 2.30 mm to (7.49, 19.1)
- moved J$1 2.30 mm to (4.64, 68.3)
- moved R1 2.30 mm to (7.49, 30.5)
- moved R2 2.30 mm to (7.52, 26.4)
Connections:
- net GND: now also IC1.AGND, IC1.GND; no longer U1.AGND, U1.GND
- net N$1: now also IC1.CD; no longer U1.CD
- net N$11: now also IC1.E8; no longer U1.E8
- net N$12: now also IC1.E9; no longer U1.E9
- net N$13: now also IC1.E10; no longer U1.E10
- net N$14: now also IC1.E11; no longer U1.E11
- net N$15: now also IC1.E12; no longer U1.E12
- net N$16: now also IC1.E15; no longer U1.E15
- net N$17: now also IC1.E16; no longer U1.E16
- net N$18: now also IC1.E17; no longer U1.E17
- net N$19: now also IC1.E18; no longer U1.E18
- net N$2: now also IC1.BUSY; no longer U1.BUSY
- net N$20: now also IC1.E19; no longer U1.E19
- net N$21: now also IC1.E20; no longer U1.E20
- net N$22: now also IC1.E21; no longer U1.E21
- net N$23: now also IC1.E22; no longer U1.E22
- net N$24: now also IC1.FS; no longer U1.FS
- net N$25: now also IC1.E13; no longer U1.E13
- net N$3: now also IC1.ANT; no longer U1.ANT
- net N$8: now also IC1.HR; no longer U1.HR
- net SDI: now also IC1.SDI; no longer U1.SDI
- net SDO: now also IC1.SDO; no longer U1.SDO
- net VCC: now also IC1.VCC; no longer U1.VCC
Routing:
- net N$25: track 36.7 -> 37.2 mm
- net N$24: track 41.7 -> 42.3 mm
Other:
- board text added: "C1"
- board text added: "R1"
- board text added: "R2"

Commit message: SMA GND schematic changes and IC name added
Parts:
- renumbered IC1 to ERIC
Changed lines of the file:
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@@
 </autorouter>
 <elements>
-<element name="IC1" library="lprs" package="ERIC" value="ERIC" x="4.6355" y="42.8625"/>
+<element name="ERIC" library="lprs" package="ERIC" value="ERIC" x="4.6355" y="42.8625"/>
 <element name="H2" library="adafruit" package="1X12-CB" value="" x="19.8755" y="18.7325" rot="R270"/>
 <element name="H1" library="adafruit" package="1X12-CB" value="" x="4.6355" y="18.7325" rot="R270"/>
@@
 <signals>
 <signal name="GND">
-<contactref element="IC1" pad="AGND"/>
+<contactref element="ERIC" pad="AGND"/>
 <contactref element="H2" pad="12"/>
 <contactref element="H2" pad="1"/>
 <contactref element="C1" pad="1"/>
-<contactref element="IC1" pad="GND"/>
+<contactref element="ERIC" pad="GND"/>
 <contactref element="H1" pad="7"/>
 <polygon width="0.4064" layer="1">
@@
 <signal name="N$1">
 <contactref element="H1" pad="1"/>
-<contactref element="IC1" pad="CD"/>
+<contactref element="ERIC" pad="CD"/>
 <wire x1="4.6355" y1="32.7025" x2="4.6355" y2="58.59245" width="0.254" layer="16"/>
 <wire x1="4.6355" y1="58.59245" x2="5.007475" y2="59.490475" width="0.254" layer="16" curve="-45"/>
@@
 <signal name="N$2">
 <contactref element="H1" pad="2"/>
-<contactref element="IC1" pad="BUSY"/>
+<contactref element="ERIC" pad="BUSY"/>
 <wire x1="4.6355" y1="30.1625" x2="5.851025" y2="31.378025" width="0.254" layer="16"/>
 <wire x1="5.851025" y1="31.378025" x2="6.223" y2="32.27605" width="0.254" layer="16" curve="45"/>
@@
 <signal name="N$3">
 <contactref element="J$1" pad="SIG"/>
-<contactref element="IC1" pad="ANT"/>
+<contactref element="ERIC" pad="ANT"/>
 <via x="7.1755" y="67.945" extent="1-16" drill="1"/>
 <wire x1="7.1755" y1="63.1825" x2="7.1755" y2="67.945" width="0.4064" layer="1"/>
@@
 <signal name="SDO">
 <contactref element="R1" pad="2"/>
-<contactref element="IC1" pad="SDO"/>
+<contactref element="ERIC" pad="SDO"/>
 <contactref element="H1" pad="3"/>
 <contactref element="R1" pad="1"/>
@@
 <contactref element="R2" pad="1"/>
 <contactref element="H1" pad="4"/>
-<contactref element="IC1" pad="SDI"/>
+<contactref element="ERIC" pad="SDI"/>
 <contactref element="R2" pad="2"/>
 <wire x1="4.6355" y1="25.0825" x2="6.428865625" y2="25.0825" width="0.254" layer="16"/>
@@
 <signal name="N$8">
 <contactref element="H1" pad="5"/>
-<contactref element="IC1" pad="HR"/>
+<contactref element="ERIC" pad="HR"/>
 <wire x1="9.398" y1="50.4825" x2="9.398" y2="25.67205" width="0.254" layer="16"/>
 <wire x1="9.398" y1="25.67205" x2="9.026025" y2="24.774025" width="0.254" layer="16" curve="-45"/>
@@
 <signal name="VCC">
 <contactref element="H1" pad="6"/>
-<contactref element="IC1" pad="VCC"/>
+<contactref element="ERIC" pad="VCC"/>
 <contactref element="C1" pad="2"/>
 <wire x1="7.493" y1="19.925" x2="7.4155" y2="20.0025" width="0.254" layer="16"/>
@@
 <signal name="N$11">
 <contactref element="H1" pad="8"/>
-<contactref element="IC1" pad="E8"/>
+<contactref element="ERIC" pad="E8"/>
 <wire x1="7.1755" y1="42.8625" x2="7.1755" y2="17.98855" width="0.254" layer="1"/>
 <wire x1="7.1755" y1="17.98855" x2="6.803525" y2="17.090525" width="0.254" layer="1" curve="-45"/>
@@
 </signal>
 <signal name="N$12">
-<contactref element="IC1" pad="E9"/>
+<contactref element="ERIC" pad="E9"/>
 <contactref element="H1" pad="9"/>
 <wire x1="9.7155" y1="42.8625" x2="9.7155" y2="42.291" width="0.254" layer="1"/>
@@
 <signal name="N$13">
 <contactref element="H1" pad="10"/>
-<contactref element="IC1" pad="E10"/>
+<contactref element="ERIC" pad="E10"/>
 <wire x1="12.2555" y1="42.8625" x2="8.563475" y2="39.170475" width="0.254" layer="1"/>
 <wire x1="8.563475" y1="39.170475" x2="8.1915" y2="38.27245" width="0.254" layer="1" curve="45"/>
@@
 </signal>
 <signal name="N$14">
-<contactref element="IC1" pad="E11"/>
+<contactref element="ERIC" pad="E11"/>
 <contactref element="H1" pad="11"/>
 <wire x1="14.7955" y1="42.8625" x2="14.360025" y2="42.8625" width="0.254" layer="1"/>
@@
 <signal name="N$15">
 <contactref element="H1" pad="12"/>
-<contactref element="IC1" pad="E12"/>
+<contactref element="ERIC" pad="E12"/>
 <wire x1="17.3355" y1="42.8625" x2="16.709525" y2="42.8625" width="0.254" layer="1"/>
 <wire x1="16.709525" y1="42.8625" x2="16.2605125" y2="42.6765125" width="0.254" layer="1" curve="45"/>
@@
 </signal>
 <signal name="N$24">
-<contactref element="IC1" pad="FS"/>
+<contactref element="ERIC" pad="FS"/>
 <contactref element="H2" pad="11"/>
 <wire x1="19.8755" y1="7.3025" x2="21.726025" y2="9.153025" width="0.254" layer="1"/>
@@
 </signal>
 <signal name="N$25">
-<contactref element="IC1" pad="E13"/>
+<contactref element="ERIC" pad="E13"/>
 <contactref element="H2" pad="10"/>
 <wire x1="19.8755" y1="9.8425" x2="21.726025" y2="11.693025" width="0.254" layer="16"/>
@@
 </signal>
 <signal name="N$16">
-<contactref element="IC1" pad="E15"/>
+<contactref element="ERIC" pad="E15"/>
 <contactref element="H2" pad="9"/>
 <wire x1="19.8755" y1="12.3825" x2="11.166975" y2="21.091025" width="0.254" layer="16"/>
@@
 <signal name="N$17">
 <contactref element="H2" pad="8"/>
-<contactref element="IC1" pad="E16"/>
+<contactref element="ERIC" pad="E16"/>
 <wire x1="19.8755" y1="14.9225" x2="12.309975" y2="22.488025" width="0.254" layer="16"/>
 <wire x1="12.309975" y1="22.488025" x2="11.938" y2="23.38605" width="0.254" layer="16" curve="-45"/>
@@
 </signal>
 <signal name="N$18">
-<contactref element="IC1" pad="E17"/>
+<contactref element="ERIC" pad="E17"/>
 <contactref element="H2" pad="7"/>
 <wire x1="19.8755" y1="17.4625" x2="13.452975" y2="23.885025" width="0.254" layer="16"/>
@@
 <signal name="N$19">
 <contactref element="H2" pad="6"/>
-<contactref element="IC1" pad="E18"/>
+<contactref element="ERIC" pad="E18"/>
 <wire x1="19.8755" y1="20.0025" x2="14.595975" y2="25.282025" width="0.254" layer="16"/>
 <wire x1="14.595975" y1="25.282025" x2="14.224" y2="26.18005" width="0.254" layer="16" curve="-45"/>
@@
 </signal>
 <signal name="N$20">
-<contactref element="IC1" pad="E19"/>
+<contactref element="ERIC" pad="E19"/>
 <contactref element="H2" pad="5"/>
 <wire x1="19.8755" y1="60.6425" x2="18.6055" y2="59.436" width="0.254" layer="1"/>
@@
 <signal name="N$21">
 <contactref element="H2" pad="4"/>
-<contactref element="IC1" pad="E20"/>
+<contactref element="ERIC" pad="E20"/>
 <wire x1="17.3355" y1="63.1825" x2="17.2085" y2="60.706" width="0.254" layer="1"/>
 <wire x1="17.2085" y1="60.706" x2="17.272" y2="25.0825" width="0.254" layer="16"/>
@@
 </signal>
 <signal name="N$22">
-<contactref element="IC1" pad="E21"/>
+<contactref element="ERIC" pad="E21"/>
 <contactref element="H2" pad="3"/>
 <wire x1="14.7955" y1="63.1825" x2="15.9385" y2="62.0395" width="0.254" layer="1"/>
@@
 </signal>
 <signal name="N$23">
-<contactref element="IC1" pad="E22"/>
+<contactref element="ERIC" pad="E22"/>
 <contactref element="H2" pad="2"/>
 <wire x1="12.2555" y1="63.1825" x2="13.97" y2="61.4045" width="0.254" layer="1"/>

Commit message: component values
Parts:
- C1: value (none) -> .1uF
- R1, R2: value (none) -> 10K
Changed lines of the file:
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@@
 <element name="H2" library="adafruit" package="1X12-CB" value="" x="19.8755" y="18.7325" rot="R270"/>
 <element name="H1" library="adafruit" package="1X12-CB" value="" x="4.6355" y="18.7325" rot="R270"/>
-<element name="R1" library="adafruit" package="R0603" value="" x="7.493" y="30.48" rot="MR270"/>
-<element name="R2" library="adafruit" package="R0603" value="" x="7.518" y="26.3525" rot="MR270"/>
-<element name="C1" library="adafruit" package="C0603K" value="" x="7.493" y="19.05" rot="MR90"/>
+<element name="R1" library="adafruit" package="R0603" value="10K" x="7.493" y="30.48" rot="MR270"/>
+<element name="R2" library="adafruit" package="R0603" value="10K" x="7.518" y="26.3525" rot="MR270"/>
+<element name="C1" library="adafruit" package="C0603K" value=".1uF" x="7.493" y="19.05" rot="MR90"/>
 <element name="J$1" library="SparkFun-Connectors" package="SMA-EDGE" value="SMA_EDGE" x="4.6355" y="68.2625"/>
 </elements>
